File: RoomSensorV2.kicad_pcb (KiCad board)
At the start: 2 copper layers, 73 x 101 mm, 17 parts, among them J1 Conn_01x02, Q1 TP0606N3-G, U1 DS3231SN#, U2 ChipCap2-SIP, U3 SeeeduinoXIAO, U4 RN2483-I_RM095

Commit message: Revision 1.0
Parts:
- added C1: 100n, Capacitor_SMD:C_0805_2012Metric, F.Cu at (93.7, 110.5)
- added C10: 1uF, Capacitor_SMD:C_0805_2012Metric, F.Cu at (88.0, 91.5)
- added C11: 100n, Capacitor_SMD:C_0805_2012Metric, F.Cu at (94.3, 97.2)
- added C2: 100n, Capacitor_SMD:C_0805_2012Metric, F.Cu at (86.1, 119.4)
- added C3: 1uF, Capacitor_SMD:C_0805_2012Metric, F.Cu at (86.7, 104.8)
- added C4: 100n, Capacitor_SMD:C_0805_2012Metric, F.Cu at (86.7, 102.9)
- added C5: 100n, Capacitor_SMD:C_0805_2012Metric, F.Cu at (79.7, 111.8)
- added C6: 4u7, Capacitor_SMD:C_0805_2012Metric, F.Cu at (77.8, 111.8)
- added C7: 4n7, Capacitor_SMD:C_0805_2012Metric, F.Cu at (102.0, 115.0)
- added C8: 10uF, Capacitor_SMD:C_0805_2012Metric, F.Cu at (80.4, 90.8)
- added C9: 10uF, Capacitor_SMD:C_0805_2012Metric, F.Cu at (88.0, 89.6)
- added D1: LED BLUE APTD2012LQBC/D, LED_SMD:LED_0805_2012Metric, F.Cu at (94.3, 104.8)
- added D2: PRTR5V0U2X,215, RoomSensorV2:SOT143B, F.Cu at (102.5, 105.0)
- added J2: Conn_01x02, Connector_PinHeader_2.54mm:PinHeader_1x02_P2.54mm_Vertical, F.Cu at (69.4, 72.8)
- added JTAG/SWD: SHF-105-01-F-D-SM, RoomSensorV2:SHF-105-01-X-D-SM, F.Cu at (108.9, 93.4)
- added R10: 300R, Resistor_SMD:R_0805_2012Metric, F.Cu at (94.3, 102.9)
- added R11: 100k, Resistor_SMD:R_0805_2012Metric, F.Cu at (94.3, 101.0)
- added R12: 1k, Resistor_SMD:R_0805_2012Metric, F.Cu at (94.3, 99.1)
- added R13: 5k1, Resistor_SMD:R_0805_2012Metric, F.Cu at (98.5, 116.9)
- added R8: 5k1, Resistor_SMD:R_0805_2012Metric, F.Cu at (98.5, 115.0)
- added R9: 1M, Resistor_SMD:R_0805_2012Metric, F.Cu at (102.0, 116.9)
- added RESET: TestPoint_2Pole, Jumper:SolderJumper-2_P1.3mm_Open_RoundedPad1.0x1.5mm, F.Cu at (93.9, 118.9)
- added U5: TC1186, Package_TO_SOT_SMD:SOT-23-5, F.Cu at (84.2, 90.8)
- added USB-C: DX07S016JA1R1500, RoomSensorV2:JAE_DX07S016JA1R1500, F.Cu at (108.3, 107.4)
- J1: value Conn_01x02 -> Conn_01x03; footprint Connector_PinHeader_2.54mm:PinHeader_1x02_P2.54mm_Vertical -> Connector_PinHeader_2.54mm:PinHeader_1x03_P2.54mm_Vertical
- R1, R2, R3: footprint Resistor_THT:R_Axial_DIN0207_L6.3mm_D2.5mm_P10.16mm_Horizontal -> Resistor_SMD:R_0805_2012Metric
- R5: value R -> 10k / 100k; footprint Resistor_THT:R_Axial_DIN0207_L6.3mm_D2.5mm_P10.16mm_Horizontal -> Resistor_SMD:R_0805_2012Metric
- R6, R7: value R -> 10k; footprint Resistor_THT:R_Axial_DIN0207_L6.3mm_D2.5mm_P10.16mm_Horizontal -> Resistor_SMD:R_0805_2012Metric
- U3: value SeeeduinoXIAO -> ATSAMD21G18A-A; footprint RoomSensorV2:SeeeduinoXIAO_SMD -> Package_QFP:TQFP-48_7x7mm_P0.5mm
- moved R5 54.4 mm to (49.9, 51.5), turned to 180 degrees
- moved R4 54.1 mm to (48.6, 47.7)
- moved U2 49.6 mm to (100.7, 61.6)
- moved J1 38.6 mm to (85.8, 72.8), turned to 90 degrees
- moved R1 37.2 mm to (71.5, 108.6), turned to 180 degrees
- moved U3 37.1 mm to (86.7, 112.4)
- moved U1 26.1 mm to (71.5, 101.6)
- moved R2 15.2 mm to (86.7, 101.0), turned to 180 degrees
- moved R3 14.3 mm to (86.7, 99.1), turned to 180 degrees
- moved Q1 12.1 mm to (72.0, 92.0), turned to 180 degrees
- moved U4 10.7 mm to (52.4, 98.5)
- moved R7 10.5 mm to (80.2, 94.1)
- moved AE1 9.32 mm to (52.4, 117.5)
- moved R6 5.76 mm to (80.2, 96.0), turned to 180 degrees
- moved BT1 0.94 mm to (77.5, 64.2)
Connections:
- J1 pad 2: VSwitched -> V_Source
- Q1 pad 1: V_Bat -> V_Source
- R1 pad 1: V_Bat -> V_Source
- R2 pad 1: I2C_SDA -> 3V3
- R2 pad 2: 3V3 -> I2C_SDA
- R3 pad 1: I2C_SCL -> 3V3
- R3 pad 2: 3V3 -> I2C_SCL
- U1 pad 14: V_Bat -> V_Source
- U3 pad 12: 3V3 -> Net-(U3-Pad12)
- U3 pad 13: GND -> Net-(U3-Pad13)
- U3 pad 15: VSwitched -> V_Bat_READ
- U3 pad 3: V_Bat_READ -> Net-(U3-Pad3)
- U3 pad 4: LIGHT_READ -> Net-(U3-Pad4)
- U3 pad 5: I2C_SDA -> GND
- U3 pad 6: I2C_SCL -> 3V3
- U3 pad 7: RN2483_UART_RX -> I2C_SDA
- U3 pad 8: RN2483_UART_TX -> I2C_SCL
- U3 pad 9: RN2483_RESET -> Net-(U3-Pad9)
Routing:
- net LIGHT_READ: track 29.6 -> 107.6 mm
- net VUSB: track 0.00 -> 70.8 mm, vias 0 -> 3
- net V_Source: track 0.00 -> 58.3 mm
- net SWDCLK: track 0.00 -> 48.5 mm, vias 0 -> 2
- net RESET: track 0.00 -> 48.4 mm, vias 0 -> 3
- net Net-(C7-Pad1): track 0.00 -> 32.9 mm
- net V_Bat_READ: track 0.00 -> 32.2 mm, vias 0 -> 4
- net VSwitched: track 75.7 -> 46.8 mm, vias 0 -> 1
- net SWDIO: track 0.00 -> 28.9 mm, vias 0 -> 2
- net Net-(D2-Pad3): track 0.00 -> 26.4 mm
- net Net-(D2-Pad2): track 0.00 -> 24.5 mm
- net V_Bat: track 50.7 -> 27.7 mm
- net RN2483_RESET: track 56.5 -> 35.8 mm, vias 2 -> 0
- net RN2483_UART_RX: track 40.4 -> 60.5 mm
- net Net-(R10-Pad1): track 0.00 -> 19.8 mm, vias 0 -> 2
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Other:
- net class Default: trace_width 0.5 -> 0.2
- net class RF added: clearance 0.2, trace_width 1, via_dia 0.8, via_drill 0.4
- board text added: "< Bat."
- board text added: "< Usb"
- board text added: "Power source select"
- board text added: "Power switch bypass"
- board text added: "SensorBoard v2.0"
- board text added: "—>"
- board text removed: "SensorBoard v1.0"
